Commit message: update test file

File: test/urdf/test_gimbal.xacro (robot description, xacro)
@@ -8,13 +8,13 @@
     <axis xyz="0 0 1"/>
   </joint>
-  <joint name="joint_pitch" type="revolute">
+  <joint name="joint_pitch" type="continuous">
     <parent link="link_yaw"/>
     <child link="link_pitch"/>
     <axis xyz="0 1 0"/>
     <origin xyz="0 0 0.25"/>
-    <limit upper="6.28" lower="-6.28" effort="1000" velocity="1000.00"/>
+    <!--    <limit lower="0.0" upper="6.0" effort="1000" velocity="1000.00"/>-->
   </joint>
   <transmission name="yaw_trans">
-    <type>transmission_interface/RevoluteTransmission</type>
+    <type>transmission_interface/SimpleTransmission</type>
     <joint name="joint_yaw">
       <offset>-0.42189619999999994</offset>
@@ -27,5 +27,5 @@
   </transmission>
   <transmission name="pitch_trans">
-    <type>transmission_interface/RevoluteTransmission</type>
+    <type>transmission_interface/SimpleTransmission</type>
     <joint name="joint_pitch">
       <offset>2.8182666160000003</offset>
