Commit message: fix configuration file

File: test/urdf/test_chassis.xacro (robot description, xacro)
@@ -1,6 +1,9 @@
 <robot name="test_robot">
   <link name="world"/>
-  <link name="link_base"/>
-  <link name="link_yaw"/>
+  <link name="base_link"/>
+  <link name="link_rf"/>
+  <link name="link_rb"/>
+  <link name="link_lf"/>
+  <link name="link_lb"/>
   <joint name="joint_rf" type="continuous">
     <parent link="base_link"/>

Commit message: test, find out stupid bug: don't update accel

File: test/urdf/test_chassis.xacro (robot description, xacro)
@@ -1,4 +1,3 @@
 <robot name="test_robot">
-  <link name="world"/>
   <link name="base_link"/>
   <link name="link_rf"/>
@@ -9,16 +8,24 @@
     <parent link="base_link"/>
     <child link="link_rf"/>
+    <origin xyz="0.38 -0.39 0"/>
+    <axis xyz="0 1 0"/>
   </joint>
   <joint name="joint_rb" type="continuous">
     <parent link="base_link"/>
     <child link="link_rb"/>
+    <origin xyz="-0.38 -0.39 0"/>
+    <axis xyz="0 1 0"/>
   </joint>
   <joint name="joint_lf" type="continuous">
     <parent link="base_link"/>
     <child link="link_lf"/>
+    <origin xyz="0.38 0.39 0"/>
+    <axis xyz="0 1 0"/>
   </joint>
   <joint name="joint_lb" type="continuous">
     <parent link="base_link"/>
     <child link="link_lb"/>
+    <origin xyz="-0.38 0.39 0"/>
+    <axis xyz="0 1 0"/>
   </joint>
   <transmission name="joint_rf_trans">
@@ -28,5 +35,5 @@
     </joint>
     <actuator name="actuator_rf">
-      <mechanicalReduction>1</mechanicalReduction>
+      <mechanicalReduction>-1</mechanicalReduction>
       <hardwareInterface>hardware_interface/EffortJointInterface</hardwareInterface>
     </actuator>
@@ -38,5 +45,5 @@
     </joint>
     <actuator name="actuator_rb">
-      <mechanicalReduction>1</mechanicalReduction>
+      <mechanicalReduction>-1</mechanicalReduction>
       <hardwareInterface>hardware_interface/EffortJointInterface</hardwareInterface>
     </actuator>
