Commit message: change word to map and change shooter param

File: test/test_shooter_with_gimbal.xacro (robot description, xacro)
@@ -1,4 +1,4 @@
 <robot name="test_robot">
-    <link name="world"/>
+    <link name="map"/>
     <link name="link_yaw"/>
     <link name="link_pitch"/>
@@ -7,5 +7,5 @@
     <link name="link_trigger"/>
     <joint name="joint_yaw" type="continuous">
-        <parent link="world"/>
+        <parent link="map"/>
         <child link="link_yaw"/>
         <axis xyz="0 0 1"/>
@@ -56,5 +56,5 @@
         <type>transmission_interface/SimpleTransmission</type>
         <joint name="joint_pitch">
-            <offset>0</offset>
+            <offset>2.7</offset>
             <hardwareInterface>hardware_interface/EffortJointInterface
             </hardwareInterface>

Commit message: update params

File: test/test_shooter_with_gimbal.xacro (robot description, xacro)
@@ -1,104 +1,104 @@
 <robot name="test_robot">
-    <link name="map"/>
-    <link name="link_yaw"/>
-    <link name="link_pitch"/>
-    <link name="link_fiction_left"/>
-    <link name="link_fiction_right"/>
-    <link name="link_trigger"/>
-    <joint name="joint_yaw" type="continuous">
-        <parent link="map"/>
-        <child link="link_yaw"/>
-        <axis xyz="0 0 1"/>
-        <origin xyz="0 0 0.12"/>
+  <link name="map"/>
+  <link name="link_yaw"/>
+  <link name="link_pitch"/>
+  <link name="link_fiction_left"/>
+  <link name="link_fiction_right"/>
+  <link name="link_trigger"/>
+  <joint name="joint_yaw" type="continuous">
+    <parent link="map"/>
+    <child link="link_yaw"/>
+    <axis xyz="0 0 1"/>
+    <origin xyz="0 0 0.153"/>
+  </joint>
+  <joint name="joint_pitch" type="continuous">
+    <parent link="link_yaw"/>
+    <child link="link_pitch"/>
+    <axis xyz="0 1 0"/>
+    <origin xyz="0 0 0.1965"/>
+    <!--    <limit lower="0.0" upper="6.0" effort="1000" velocity="1000.00"/>-->
+  </joint>
+  <joint name="joint_fiction_left" type="continuous">
+    <parent link="link_pitch"/>
+    <child link="link_fiction_left"/>
+    <axis xyz="0 1 0"/>
+    <origin xyz="0 0 0.25"/>
+    <!--<limit upper="6.28" lower="-6.28" effort="1000" velocity="1000.00"/>-->
+  </joint>
+  <joint name="joint_fiction_right" type="continuous">
+    <parent link="link_pitch"/>
+    <child link="link_fiction_right"/>
+    <axis xyz="0 1 0"/>
+    <origin xyz="0 0 0.25"/>
+    <!--<limit upper="6.28" lower="-6.28" effort="1000" velocity="1000.00"/>-->
+  </joint>
+  <joint name="joint_trigger" type="continuous">
+    <parent link="link_pitch"/>
+    <child link="link_trigger"/>
+    <axis xyz="0 1 0"/>
+    <origin xyz="0 0 0.25"/>
+    <!--<limit upper="6.28" lower="-6.28" effort="1000" velocity="1000.00"/>-->
+  </joint>
+  <transmission name="yaw_trans">
+    <type>transmission_interface/SimpleTransmission</type>
+    <joint name="joint_yaw">
+      <offset>0.4096</offset>
+      <hardwareInterface>hardware_interface/EffortJointInterface
+      </hardwareInterface>
     </joint>
-    <joint name="joint_pitch" type="continuous">
-        <parent link="link_yaw"/>
-        <child link="link_pitch"/>
-        <axis xyz="0 1 0"/>
-        <origin xyz="0 0 0.1965"/>
-        <!--    <limit lower="0.0" upper="6.0" effort="1000" velocity="1000.00"/>-->
+    <actuator name="actuator_yaw">
+      <mechanicalReduction>1</mechanicalReduction>
+      <hardwareInterface>hardware_interface/EffortJointInterface
+      </hardwareInterface>
+    </actuator>
+  </transmission>
+  <transmission name="pitch_trans">
+    <type>transmission_interface/SimpleTransmission</type>
+    <joint name="joint_pitch">
+      <offset>2.7</offset>
+      <hardwareInterface>hardware_interface/EffortJointInterface
+      </hardwareInterface>
     </joint>
-    <joint name="joint_fiction_left" type="continuous">
-        <parent link="link_pitch"/>
-        <child link="link_fiction_left"/>
-        <axis xyz="0 1 0"/>
-        <origin xyz="0 0 0.25"/>
-        <!--<limit upper="6.28" lower="-6.28" effort="1000" velocity="1000.00"/>-->
+    <actuator name="actuator_pitch">
+      <mechanicalReduction>-1</mechanicalReduction>
+      <hardwareInterface>hardware_interface/EffortJointInterface
+      </hardwareInterface>
+    </actuator>
+  </transmission>
+  <transmission name="fiction_left_trans">
+    <type>transmission_interface/SimpleTransmission</type>
+    <joint name="joint_fiction_left">
+      <hardwareInterface>hardware_interface/EffortJointInterface
+      </hardwareInterface>
     </joint>
-    <joint name="joint_fiction_right" type="continuous">
-        <parent link="link_pitch"/>
-        <child link="link_fiction_right"/>
-        <axis xyz="0 1 0"/>
-        <origin xyz="0 0 0.25"/>
-        <!--<limit upper="6.28" lower="-6.28" effort="1000" velocity="1000.00"/>-->
+    <actuator name="actuator_fiction_left">
+      <mechanicalReduction>-1</mechanicalReduction>
+      <hardwareInterface>hardware_interface/EffortJointInterface
+      </hardwareInterface>
+    </actuator>
+  </transmission>
+  <transmission name="fiction_right_trans">
+    <type>transmission_interface/SimpleTransmission</type>
+    <joint name="joint_fiction_right">
+      <hardwareInterface>hardware_interface/EffortJointInterface
+      </hardwareInterface>
     </joint>
-    <joint name="joint_trigger" type="continuous">
-        <parent link="link_pitch"/>
-        <child link="link_trigger"/>
-        <axis xyz="0 1 0"/>
-        <origin xyz="0 0 0.25"/>
-        <!--<limit upper="6.28" lower="-6.28" effort="1000" velocity="1000.00"/>-->
+    <actuator name="actuator_fiction_right">
+      <mechanicalReduction>1</mechanicalReduction>
+      <hardwareInterface>hardware_interface/EffortJointInterface
+      </hardwareInterface>
+    </actuator>
+  </transmission>
+  <transmission name="trigger_trans">
+    <type>transmission_interface/SimpleTransmission</type>
+    <joint name="joint_trigger">
+      <hardwareInterface>hardware_interface/EffortJointInterface
+      </hardwareInterface>
     </joint>
-    <transmission name="yaw_trans">
-        <type>transmission_interface/SimpleTransmission</type>
-        <joint name="joint_yaw">
-            <offset>0.4096</offset>
-            <hardwareInterface>hardware_interface/EffortJointInterface
-            </hardwareInterface>
-        </joint>
-        <actuator name="actuator_yaw">
-            <mechanicalReduction>1</mechanicalReduction>
-            <hardwareInterface>hardware_interface/EffortJointInterface
-            </hardwareInterface>
-        </actuator>
-    </transmission>
-    <transmission name="pitch_trans">
-        <type>transmission_interface/SimpleTransmission</type>
-        <joint name="joint_pitch">
-            <offset>2.7</offset>
-            <hardwareInterface>hardware_interface/EffortJointInterface
-            </hardwareInterface>
-        </joint>
-        <actuator name="actuator_pitch">
-            <mechanicalReduction>-1</mechanicalReduction>
-            <hardwareInterface>hardware_interface/EffortJointInterface
-            </hardwareInterface>
-        </actuator>
-    </transmission>
-    <transmission name="fiction_left_trans">
-        <type>transmission_interface/SimpleTransmission</type>
-        <joint name="joint_fiction_left">
-            <hardwareInterface>hardware_interface/EffortJointInterface
-            </hardwareInterface>
-        </joint>
-        <actuator name="actuator_fiction_left">
-            <mechanicalReduction>-1</mechanicalReduction>
-            <hardwareInterface>hardware_interface/EffortJointInterface
-            </hardwareInterface>
-        </actuator>
-    </transmission>
-    <transmission name="fiction_right_trans">
-        <type>transmission_interface/SimpleTransmission</type>
-        <joint name="joint_fiction_right">
-            <hardwareInterface>hardware_interface/EffortJointInterface
-            </hardwareInterface>
-        </joint>
-        <actuator name="actuator_fiction_right">
-            <mechanicalReduction>1</mechanicalReduction>
-            <hardwareInterface>hardware_interface/EffortJointInterface
-            </hardwareInterface>
-        </actuator>
-    </transmission>
-    <transmission name="trigger_trans">
-        <type>transmission_interface/SimpleTransmission</type>
-        <joint name="joint_trigger">
-            <hardwareInterface>hardware_interface/EffortJointInterface
-            </hardwareInterface>
-        </joint>
-        <actuator name="actuator_trigger">
-            <mechanicalReduction>-1</mechanicalReduction>
-            <hardwareInterface>hardware_interface/EffortJointInterface
-            </hardwareInterface>
-        </actuator>
-    </transmission>
+    <actuator name="actuator_trigger">
+      <mechanicalReduction>-1</mechanicalReduction>
+      <hardwareInterface>hardware_interface/EffortJointInterface
+      </hardwareInterface>
+    </actuator>
+  </transmission>
 </robot>

Commit message: update parameter

File: test/test_shooter_with_gimbal.xacro (robot description, xacro)
@@ -10,5 +10,5 @@
         <child link="link_yaw"/>
         <axis xyz="0 0 1"/>
-        <origin xyz="0 0 0.12"/>
+        <origin xyz="0 0 0.16"/>
     </joint>
     <joint name="joint_pitch" type="continuous">
