Commit message: change word to map and change shooter param

File: test/test_gimbal.xacro (robot description, xacro)
@@ -1,8 +1,8 @@
 <robot name="test_robot">
-  <link name="world"/>
+  <link name="map"/>
   <link name="link_yaw"/>
   <link name="link_pitch"/>
   <joint name="joint_yaw" type="continuous">
-    <parent link="world"/>
+    <parent link="map"/>
     <child link="link_yaw"/>
     <axis xyz="0 0 1"/>
@@ -18,5 +18,5 @@
     <type>transmission_interface/SimpleTransmission</type>
     <joint name="joint_yaw">
-      <offset>0.4</offset>
+      <offset>0.0</offset>
       <hardwareInterface>hardware_interface/EffortJointInterface</hardwareInterface>
     </joint>

Commit message: update parameter

File: test/test_gimbal.xacro (robot description, xacro)
@@ -7,4 +7,5 @@
     <child link="link_yaw"/>
     <axis xyz="0 0 1"/>
+    <origin xyz="0 0 0.16"/>
   </joint>
   <joint name="joint_pitch" type="continuous">
@@ -12,5 +13,5 @@
     <child link="link_pitch"/>
     <axis xyz="0 1 0"/>
-    <origin xyz="0 0 0.25"/>
+    <origin xyz="0 0 0.1925"/>
     <!--    <limit lower="0.0" upper="6.0" effort="1000" velocity="1000.00"/>-->
   </joint>
@@ -18,5 +19,5 @@
     <type>transmission_interface/SimpleTransmission</type>
     <joint name="joint_yaw">
-      <offset>0.0</offset>
+      <offset>0.4096</offset>
       <hardwareInterface>hardware_interface/EffortJointInterface</hardwareInterface>
     </joint>
@@ -29,5 +30,5 @@
     <type>transmission_interface/SimpleTransmission</type>
     <joint name="joint_pitch">
-      <offset>2.8182666160000003</offset>
+      <offset>2.7</offset>
       <hardwareInterface>hardware_interface/EffortJointInterface</hardwareInterface>
     </joint>
